File: decode.kicad_sch (KiCad schematic)
At the start: 13 parts, among them J10 Conn_01x01_Female, J13 Conn_01x01_Female, J14 Conn_01x01_Female, J15 Conn_01x01_Female, J16 Conn_01x01_Female, J9 Conn_01x01_Female, U5 74HC00, U6 74LS139

Commit message: Add files via upload
Parts:
- removed J10, J13, J14, J15, J16, J9: Conn_01x01_Female, Connector_PinHeader_2.00mm:PinHeader_1x01_P2.00mm_Vertical, symbol Connector:Conn_01x01_Female
- removed unit 1 of U5
- added U1: 74HC00, symbol 74xx:74HC00
- added U7: 74HC00, Package_DIP:DIP-14_W7.62mm, symbol 74xx:74HC00
- renumbered C8 to C3, C9 to C4, D2 to D1, R4 to R1, R5 to R2, U6 to U10, U5 to U9
Connections:
- net A12: now also U10.3 (A1)
- net E: now also U7.1
- net BSEL2*: now reaches U10.6 (O2)
- net at U10.7 (O3): now also U1.1, U1.2
- net BSEL* renamed BSEL0*
- net IOSEL* renamed BSEL1*
- new net: U1.3, U7.2
- new net GSEL*: U7.3
Other:
- note added: "C000-C7FF"
- note added: "C800-CFFF"
- note added: "Memory Map: 0000-7FFF volatile SRAM 32k 8000-BFFF NVRAM bank 0/1 16k C000-C7FF select not assigned 2K C800-CFFF select not assigned 2K D000-D7FF main bus select 2K D800-DFFF onboard peripheral select 2K E000-FFFF EEPROM 8K"
- note removed: "Memory Map: 0000-7FFF volatile SRAM 32k 8000-BFFF NVRAM bank 0/1 16k C000-CFFF not assigned 4K D000-D7FF main bus select 2K D800-DFFF I/O bus select 2K E000-FFFF EEPROM 8K"
